File: output/pcbs/base.kicad_pcb (KiCad board)
At the start: 2 copper layers, 282.4 x 115.1 mm, 116 parts

Commit message: final version... for now
Parts:
- removed the ? at (218.0, 81.8)
- removed the ? at (321.3, 106.0)
- removed the ? at (243.0, 81.8)
- removed the ? at (139.6, 106.0)
- added ?: , HOLE_M2_TH, F.Cu at (223.0, 95.3)
- added ?: , HOLE_M2_TH, F.Cu at (288.0, 127.5)
- added ?: , HOLE_M2_TH, F.Cu at (238.0, 95.3)
- added ?: , HOLE_M2_TH, F.Cu at (218.0, 34.5)
- added ?: , HOLE_M2_TH, F.Cu at (243.0, 34.5)
- added ?: , HOLE_M2_TH, F.Cu at (124.3, 109.2)
- added ?: , HOLE_M2_TH, F.Cu at (336.6, 109.2)
- added ?: , HOLE_M2_TH, F.Cu at (101.3, 28.3)
- added ?: , HOLE_M2_TH, F.Cu at (359.7, 28.3)
- added ?: , HOLE_M2_TH, F.Cu at (172.9, 127.5)
Routing:
- net P111: track 447.6 -> 0.00 mm, vias 22 -> 0
- net P106: track 431.2 -> 0.00 mm, vias 18 -> 0
- net P011: track 428.0 -> 0.00 mm, vias 4 -> 0
- net P104: track 411.2 -> 0.00 mm, vias 16 -> 0
- net P010: track 351.7 -> 0.00 mm, vias 18 -> 0
- net P009: track 230.4 -> 0.00 mm, vias 10 -> 0
- net P024: track 181.5 -> 0.00 mm
- net P115: track 178.5 -> 0.00 mm
- net P002: track 156.7 -> 0.00 mm
- net P020: track 150.7 -> 0.00 mm
- net P022: track 150.4 -> 0.00 mm, vias 2 -> 0
- net P100: track 143.0 -> 0.00 mm
- net P113: track 136.7 -> 0.00 mm
- net P029: track 136.3 -> 0.00 mm
- net P031: track 134.4 -> 0.00 mm
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- removed copper zone on B.Cu, net (none)
- removed copper zone on F.Cu, net (none)
Other:
- outline, holes or cut-outs redrawn
- net class Default added: clearance 0.2, trace_width 0.25, via_dia 0.8, via_drill 0.4
- board text removed: "centiwati-hugging"
- board text removed: "chasm"
